File: x68030_scsi/x68030_scsi.kicad_pcb (KiCad board)
At the start: 2 copper layers, 41 parts, among them J1 Conn_02x25_Odd_Even, J2 Conn_02x20_Odd_Even, SW1 SW_DIP_x03

Commit message: Update
Parts:
- removed SW1: SW_DIP_x03, Button_Switch_SMD:SW_DIP_SPSTx03_Slide_Omron_A6S-310x_W8.9mm_P2.54mm
- added H1: MountingHole, MountingHole:MountingHole_4.3mm_M4, F.Cu at (41.0, 88.0)
- added H2: MountingHole, MountingHole:MountingHole_4.3mm_M4, F.Cu at (41.0, 170.0)
- added J3: Conn_02x03_Odd_Even, Connector_PinHeader_2.54mm:PinHeader_2x03_P2.54mm_Vertical, F.Cu at (37.0, 146.0)
- moved R11 88.3 mm to (42.1, 136.9)
- moved R12 88.3 mm to (42.1, 139.4)
- moved R14 88.3 mm to (42.1, 144.5)
- moved R15 88.3 mm to (42.1, 147.0)
- moved R17 88.3 mm to (42.1, 152.0)
- moved R18 88.3 mm to (42.1, 154.5)
- moved R13 88.3 mm to (42.1, 141.9)
- moved R16 88.3 mm to (42.1, 149.5)
- moved F1 78.9 mm to (37.6, 111.5)
- moved R1 78.1 mm to (42.1, 111.9)
- moved R10 78.1 mm to (42.1, 134.5)
- moved R2 78.1 mm to (42.1, 114.4)
- moved R3 78.1 mm to (42.1, 116.9)
- moved R4 78.1 mm to (42.1, 119.4)
- moved R5 78.1 mm to (42.1, 122.0)
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Connections:
- C1 pad 1: Net-(C1-Pad1) -> /DB0
- C10 pad 1: Net-(C10-Pad1) -> //ATN
- C11 pad 1: Net-(C11-Pad1) -> //BSY
- C12 pad 1: Net-(C12-Pad1) -> //ACK
- C13 pad 1: Net-(C13-Pad1) -> //RST
- C14 pad 1: Net-(C14-Pad1) -> //MSG
- C15 pad 1: Net-(C15-Pad1) -> //SEL
- C16 pad 1: Net-(C16-Pad1) -> //I/O
- C17 pad 1: Net-(C17-Pad1) -> //C/D
- C18 pad 1: Net-(C18-Pad1) -> //REQ
- C2 pad 1: Net-(C2-Pad1) -> /DB1
- C3 pad 1: Net-(C3-Pad1) -> /DB2
- C4 pad 1: Net-(C4-Pad1) -> /DB3
- C5 pad 1: Net-(C5-Pad1) -> /DB4
- C6 pad 1: Net-(C6-Pad1) -> /DB5
- C7 pad 1: Net-(C7-Pad1) -> /DB6
- C8 pad 1: Net-(C8-Pad1) -> /DB7
- C9 pad 1: Net-(C9-Pad1) -> /PARITY
- J2 pad 1: unconnected-(J2-Pin_1-Pad1) -> /ID_SWITCH1
- J2 pad 10: unconnected-(J2-Pin_10-Pad10) -> /DB1
- J2 pad 12: unconnected-(J2-Pin_12-Pad12) -> /DB2
- J2 pad 14: unconnected-(J2-Pin_14-Pad14) -> /DB3
- J2 pad 16: unconnected-(J2-Pin_16-Pad16) -> /DB4
- J2 pad 18: unconnected-(J2-Pin_18-Pad18) -> /DB5
- J2 pad 19: unconnected-(J2-Pin_19-Pad19) -> /DB6
- J2 pad 2: unconnected-(J2-Pin_2-Pad2) -> /ID_SWITCH2
- J2 pad 21: unconnected-(J2-Pin_21-Pad21) -> /DB7
- J2 pad 23: unconnected-(J2-Pin_23-Pad23) -> /PARITY
- J2 pad 26: unconnected-(J2-Pin_26-Pad26) -> //ATN
- J2 pad 27: unconnected-(J2-Pin_27-Pad27) -> //BSY
- J2 pad 29: unconnected-(J2-Pin_29-Pad29) -> //ACK
- J2 pad 3: unconnected-(J2-Pin_3-Pad3) -> /ID_SWITCH3
- J2 pad 30: unconnected-(J2-Pin_30-Pad30) -> //RST
- J2 pad 31: unconnected-(J2-Pin_31-Pad31) -> //MSG
- J2 pad 33: unconnected-(J2-Pin_33-Pad33) -> //SEL
- J2 pad 34: unconnected-(J2-Pin_34-Pad34) -> //I/O
- J2 pad 35: unconnected-(J2-Pin_35-Pad35) -> //C/D
- J2 pad 37: unconnected-(J2-Pin_37-Pad37) -> //REQ
- J2 pad 8: unconnected-(J2-Pin_8-Pad8) -> /DB0
- R1 pad 2: Net-(C1-Pad1) -> /DB0
- R10 pad 2: Net-(C10-Pad1) -> //ATN
- R11 pad 2: Net-(C11-Pad1) -> //BSY
- R12 pad 2: Net-(C12-Pad1) -> //ACK
- R13 pad 2: Net-(C13-Pad1) -> //RST
- R14 pad 2: Net-(C14-Pad1) -> //MSG
- R15 pad 2: Net-(C15-Pad1) -> //SEL
- R16 pad 2: Net-(C16-Pad1) -> //I/O
- R17 pad 2: Net-(C17-Pad1) -> //C/D
- R18 pad 2: Net-(C18-Pad1) -> //REQ
- R2 pad 2: Net-(C2-Pad1) -> /DB1
- R3 pad 2: Net-(C3-Pad1) -> /DB2
- R4 pad 2: Net-(C4-Pad1) -> /DB3
- R5 pad 2: Net-(C5-Pad1) -> /DB4
- R6 pad 2: Net-(C6-Pad1) -> /DB5
- R7 pad 2: Net-(C7-Pad1) -> /DB6
- R8 pad 2: Net-(C8-Pad1) -> /DB7
- R9 pad 2: Net-(C9-Pad1) -> /PARITY
Routing:
- net //REQ: track 0.00 -> 123.9 mm
- net //I/O: track 0.00 -> 123.6 mm, vias 0 -> 3
- net //C/D: track 0.00 -> 115.0 mm
- net //SEL: track 0.00 -> 106.2 mm
- net //MSG: track 0.00 -> 101.3 mm
- net //RST: track 0.00 -> 99.9 mm
- net //ACK: track 0.00 -> 94.6 mm
- net //BSY: track 0.00 -> 91.2 mm
- net //ATN: track 0.00 -> 90.9 mm, vias 0 -> 1
- net /ID_SWITCH2: track 0.00 -> 89.3 mm
- net /ID_SWITCH1: track 0.00 -> 80.1 mm
- net /PARITY: track 0.00 -> 73.2 mm, vias 0 -> 1
- net /DB7: track 0.00 -> 71.2 mm, vias 0 -> 1
- net /DB3: track 0.00 -> 69.9 mm, vias 0 -> 1
- net /DB1: track 0.00 -> 69.8 mm, vias 0 -> 1
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- added copper zone on B.Cu, net GND
- added copper zone on F.Cu, net GND
Other:
- board outline added: 56 x 105 mm
- board text added: "0"
- board text added: "1"
- board text added: "2"
- board text added: "IDSW"
- board text added: "JLCJLCJLCJLC"
- board text added: "X68030 SCSI ADAPTER"
- board text added: "buffi 2025"

Commit message: fixes
Parts:
- removed JP1: Jumper_2_Open, Resistor_SMD:R_0603_1608Metric_Pad0.98x0.95mm_HandSolder
- removed R1, R10, R11, R12, R13, R14, R15, R16, R17, R18, R2, R3, R4, R5, R6, R7, R8, R9: R_Small_US, Resistor_SMD:R_0603_1608Metric_Pad0.98x0.95mm_HandSolder
- added J5: Conn_01x04, Connector_PinHeader_2.54mm:PinHeader_1x04_P2.54mm_Horizontal, F.Cu at (72.8, 84.5)
- added RN1: 4611X-104-221/331L, Resistor_THT:R_Array_SIP11, F.Cu at (38.9, 95.2)
- added RN2: 4611X-104-221/331L, Resistor_THT:R_Array_SIP11, F.Cu at (38.9, 138.2)
- C1, C10, C11, C12, C13, C14, C15, C16, C17, C18, C2, C3, C4, C5, C6, C7, C8, C9: value C_Small -> 47p; footprint Capacitor_SMD:C_0603_1608Metric_Pad1.08x0.95mm_HandSolder -> Capacitor_SMD:C_0805_2012Metric_Pad1.18x1.45mm_HandSolder
- F1: value Fuse -> 1A; footprint Fuse:Fuse_0603_1608Metric_Pad1.05x0.95mm_HandSolder -> Fuse:Fuse_0805_2012Metric_Pad1.15x1.40mm_HandSolder
- J1: value Conn_02x25_Odd_Even -> Internal SCSI
- J2: value Conn_02x20_Odd_Even -> X68030 SCSI
- moved C18 82.0 mm to (61.5, 165.1), turned to 0 degrees
- moved C17 79.0 mm to (61.5, 162.6), turned to 0 degrees
- moved C16 76.0 mm to (61.5, 160.0), turned to 0 degrees
- moved C15 73.2 mm to (61.5, 157.5), turned to 0 degrees
- moved C14 70.3 mm to (61.5, 154.9), turned to 0 degrees
- moved C13 67.6 mm to (61.5, 152.4), turned to 0 degrees
- moved C12 64.9 mm to (61.5, 149.9), turned to 0 degrees
- moved C11 62.3 mm to (61.5, 147.3), turned to 0 degrees
- moved C10 57.4 mm to (61.5, 142.2), turned to 0 degrees
- moved C9 39.9 mm to (61.5, 124.5), turned to 0 degrees
- moved C8 37.8 mm to (61.5, 121.9), turned to 0 degrees
- moved C7 36.0 mm to (61.5, 119.4), turned to 0 degrees
- moved C6 34.3 mm to (61.5, 116.8), turned to 0 degrees
- moved C5 32.9 mm to (61.5, 114.3), turned to 0 degrees
- moved C1 26.0 mm to (61.5, 104.0), turned to 0 degrees
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Connections:
- net /ID_SWITCH1 renamed /ID0
- net /ID_SWITCH2 renamed /ID1
- net /ID_SWITCH3 renamed /ID2
- C16 pad 1: //I/O -> //C/D
- C17 pad 1: //C/D -> //REQ
- C18 pad 1: //REQ -> //I/O
- F1 pad 1: VCC -> /TMPWR
- F1 pad 2: Net-(F1-Pad2) -> Net-(J2-Pin_25)
- J2 pad 11: unconnected-(J2-Pin_11-Pad11) -> GND
- J2 pad 13: unconnected-(J2-Pin_13-Pad13) -> GND
- J2 pad 15: unconnected-(J2-Pin_15-Pad15) -> GND
- J2 pad 17: unconnected-(J2-Pin_17-Pad17) -> GND
- J2 pad 25: VCC -> Net-(J2-Pin_25)
- J2 pad 39: /NO_IDEA2 -> /VCC1
- J2 pad 4: unconnected-(J2-Pin_4-Pad4) -> /HDLED
- J2 pad 40: /NO_IDEA2 -> /VCC1
- J2 pad 5: /NO_IDEA1 -> /VCC1
- J2 pad 6: /NO_IDEA1 -> /VCC1
- J2 pad 7: unconnected-(J2-Pin_7-Pad7) -> GND
- J2 pad 9: unconnected-(J2-Pin_9-Pad9) -> GND
Routing:
- net /TMPWR: track 0.00 -> 76.8 mm
- net VCC: track 63.5 -> 0.00 mm, vias 1 -> 0
- net /HDLED: track 0.00 -> 57.7 mm
- net /VCC1: track 0.00 -> 51.5 mm
- net Net-(F1-Pad2): track 45.6 -> 0.00 mm
- net /NO_IDEA1: track 42.4 -> 0.00 mm, vias 1 -> 0
- net Net-(J2-Pin_25): track 0.00 -> 36.1 mm
- net /ID1: track 89.3 -> 60.3 mm
- net /ID0: track 80.1 -> 58.2 mm
- net /DB1: track 69.8 -> 52.1 mm, vias 1 -> 0
- net /ID2: track 67.1 -> 51.2 mm
- net //I/O: track 123.6 -> 138.8 mm, vias 3 -> 0
- net /DB2: track 67.7 -> 55.3 mm, vias 1 -> 0
- net /DB3: track 69.9 -> 58.6 mm, vias 1 -> 0
- net /DB0: track 59.1 -> 49.8 mm
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Other:
- outline, holes or cut-outs redrawn

Commit message: Update x68030_scsi.kicad_pcb
Routing:
- net /ID1: track 60.3 -> 72.8 mm
- net /ID0: track 58.2 -> 56.1 mm
Other:
- board text added: "39"
- board text added: "40"
- board text added: "GND"
- board text added: "HDLED"
- board text added: "VCC"
