File: x68030_scsi/x68030_scsi.kicad_pcb (KiCad board)
At the start: 2 copper layers, 56 x 105 mm, 27 parts, among them J1 Internal SCSI, J2 X68030 SCSI, J3 Conn_02x03_Odd_Even, J5 Conn_01x04

Commit message: misc
Parts:
- moved J3 4.32 mm to (43.4, 131.8)
Routing:
- net /ID2: track 51.2 -> 55.6 mm
- net /ID0: track 56.1 -> 59.5 mm
Changed lines of the file:
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@@
 	(footprint "Connector_PinHeader_2.54mm:PinHeader_2x03_P2.54mm_Vertical"
 		(layer "F.Cu")
-		(at 39.116 131.826 180)
+		(at 43.439 131.811 180)
 		(descr "Through hole straight pin header, 2x03, 2.54mm pitch, double rows")
 		(tags "Through hole pin header THT 2x03 2.54mm double row")
@@
 	)
 	(gr_text "0"
-		(at 33.576 132.246 0)
+		(at 37.338 132.334 0)
 		(layer "F.SilkS")
 		(effects
@@
 	)
 	(gr_text "1"
-		(at 33.576 129.746 0)
+		(at 37.338 129.834 0)
 		(layer "F.SilkS")
 		(effects
@@
 	)
 	(gr_text "IDSW"
-		(at 42.926 131.191 90)
+		(at 40.386 124.587 0)
 		(layer "F.SilkS")
 		(effects
@@
 	)
 	(gr_text "2"
-		(at 33.576 127.246 0)
+		(at 37.338 127.334 0)
 		(layer "F.SilkS")
 		(effects
@@
 	)
 	(segment
-		(start 41.529 133.096)
-		(end 41.529 130.302)
+		(start 45.212 133.35)
+		(end 44.577 133.985)
 		(width 0.25)
 		(layer "B.Cu")
@@
 	)
 	(segment
-		(start 33.655 131.953)
-		(end 35.814 134.112)
+		(start 43.439 129.271)
+		(end 44.181 129.271)
 		(width 0.25)
 		(layer "B.Cu")
@@
 	)
 	(segment
-		(start 38.5 76)
-		(end 33.655 80.845)
+		(start 33.655 80.845)
+		(end 38.5 76)
 		(width 0.25)
 		(layer "B.Cu")
@@
 	)
 	(segment
-		(start 40.513 129.286)
-		(end 39.116 129.286)
+		(start 33.655 127.127)
+		(end 33.655 80.845)
 		(width 0.25)
 		(layer "B.Cu")
@@
 	)
 	(segment
-		(start 41.529 130.302)
-		(end 40.513 129.286)
+		(start 44.181 129.271)
+		(end 45.212 130.302)
 		(width 0.25)
 		(layer "B.Cu")
@@
 	)
 	(segment
-		(start 35.814 134.112)
-		(end 40.513 134.112)
+		(start 45.212 130.302)
+		(end 45.212 133.35)
 		(width 0.25)
 		(layer "B.Cu")
@@
 	)
 	(segment
-		(start 33.655 80.845)
-		(end 33.655 131.953)
+		(start 44.577 133.985)
+		(end 40.513 133.985)
 		(width 0.25)
 		(layer "B.Cu")
@@
 	)
 	(segment
-		(start 40.513 134.112)
-		(end 41.529 133.096)
+		(start 40.513 133.985)
+		(end 33.655 127.127)
 		(width 0.25)
 		(layer "B.Cu")
@@
 	(segment
 		(start 40.5 80.658)
-		(end 40.5 78)
+		(end 36.83 84.328)
 		(width 0.25)
 		(layer "B.Cu")
@@
 	)
 	(segment
-		(start 36.83 84.328)
-		(end 40.5 80.658)
+		(start 38.608 125.222)
+		(end 43.053 125.222)
+		(width 0.25)
+		(layer "B.Cu")
+		(net 26)
+	)
+	(segment
+		(start 36.83 123.444)
+		(end 38.608 125.222)
+		(width 0.25)
+		(layer "B.Cu")
+		(net 26)
+	)
+	(segment
+		(start 43.053 125.222)
+		(end 43.439 125.608)
 		(width 0.25)
 		(layer "B.Cu")
@@
 	)
 	(segment
-		(start 39.116 125.73)
+		(start 36.83 84.328)
 		(end 36.83 123.444)
 		(width 0.25)
@@
 	)
 	(segment
-		(start 36.83 123.444)
-		(end 36.83 84.328)
+		(start 40.5 78)
+		(end 40.5 80.658)
 		(width 0.25)
 		(layer "B.Cu")
@@
 	)
 	(segment
-		(start 39.116 126.746)
-		(end 39.116 125.73)
+		(start 43.439 125.608)
+		(end 43.439 126.731)
 		(width 0.25)
 		(layer "B.Cu")
@@
 	)
 	(segment
-		(start 37.846 125.984)
-		(end 36.068 124.206)
+		(start 42.184 130.556)
+		(end 39.37 130.556)
 		(width 0.25)
 		(layer "B.Cu")
@@
 	)
 	(segment
-		(start 36.068 80.432)
-		(end 38.5 78)
+		(start 36.068 127.254)
+		(end 36.068 80.432)
 		(width 0.25)
 		(layer "B.Cu")
@@
 	)
 	(segment
-		(start 37.846 130.556)
-		(end 37.846 125.984)
+		(start 43.439 131.811)
+		(end 42.184 130.556)
 		(width 0.25)
 		(layer "B.Cu")
@@
 	)
 	(segment
-		(start 39.116 131.826)
-		(end 37.846 130.556)
+		(start 39.37 130.556)
+		(end 36.068 127.254)
 		(width 0.25)
 		(layer "B.Cu")
@@
 	)
 	(segment
-		(start 36.068 124.206)
-		(end 36.068 80.432)
+		(start 36.068 80.432)
+		(end 38.5 78)
 		(width 0.25)
 		(layer "B.Cu")

Commit message: fix stuff
Parts:
- removed J3: Conn_02x03_Odd_Even, Connector_PinHeader_2.54mm:PinHeader_2x03_P2.54mm_Vertical
- removed J5: Conn_01x04, Connector_PinHeader_2.54mm:PinHeader_1x04_P2.54mm_Horizontal
- added JP1: Jumper_2_Small_Bridged, Jumper:SolderJumper-2_P1.3mm_Bridged_Pad1.0x1.5mm, B.Cu at (73.4, 90.9)
- added TP1: EXTERNAL_HDLED1, TestPoint:TestPoint_Pad_1.5x1.5mm, B.Cu at (81.8, 91.9)
- added U2: 74LVC1G07, Package_TO_SOT_SMD:SOT-23-5_HandSoldering, F.Cu at (76.7, 85.6)
Connections:
- J2 pad 4: /HDLED -> /HDLED-
Routing:
- net /ID1: track 73.0 -> 0.00 mm
- net /ID0: track 59.5 -> 0.00 mm
- net /HDLED: track 57.7 -> 0.00 mm
- net /ID2: track 55.6 -> 0.00 mm
- net /HDLED-: track 0.00 -> 52.4 mm
- net //BSY: track 97.4 -> 110.0 mm, vias 0 -> 2
- net Net-(JP1-A): track 0.00 -> 12.2 mm, vias 0 -> 1
- net /VCC1: track 51.3 -> 49.2 mm
Other:
- board text removed: "0"
- board text removed: "GND"
- board text removed: "HDLED"
- board text removed: "IDSW"
- board text removed: "VCC"
