File: x68030_scsi/x68030_scsi.kicad_pcb (KiCad board)
At the start: 2 copper layers, 56 x 105 mm, 28 parts, among them J1 Internal SCSI, J2 X68030 SCSI, U2 74LVC1G07

Commit message: updates
Parts:
- removed TP1: EXTERNAL_HDLED1, TestPoint:TestPoint_Pad_1.5x1.5mm
- removed U2: 74LVC1G07, Package_TO_SOT_SMD:SOT-23-5_HandSoldering
- added J3: Conn_01x02, Connector_JST:JST_XH_B2B-XH-A_1x02_P2.50mm_Vertical, F.Cu at (80.1, 88.5)
- added JP2: Jumper_2_Open, Jumper:SolderJumper-2_P1.3mm_Open_Pad1.0x1.5mm, B.Cu at (82.7, 80.7)
- added U1: SN74LVC1G14DBV, Package_TO_SOT_SMD:SOT-23-5, F.Cu at (73.8, 90.4)
- JP1: value Jumper_2_Small_Bridged -> Jumper_2_Bridged
- moved JP1 16.1 mm to (82.7, 77.8), turned to 0 degrees
Connections:
- JP1 pad 2: //BSY -> /HDLED-
Routing:
- net Net-(J3-Pin_1): track 0.00 -> 14.4 mm
- net //BSY: track 110.0 -> 97.4 mm, vias 2 -> 0
- net /VCC1: track 49.2 -> 55.4 mm
- net Net-(J3-Pin_2): track 0.00 -> 6.14 mm
- net Net-(JP1-A): track 12.2 -> 14.5 mm
- net /HDLED-: track 52.4 -> 52.9 mm, vias 0 -> 1
Other:
- board text added: "(-)"
- board text added: "+"
- board text added: "HDLED"
- board text added: "github.com/buffis/x68030_scsi_adapter"
