File: x68030_scsi/x68030_scsi.kicad_sch (KiCad schematic)
At the start: 41 parts

Commit message: misc
Parts:
- C1, C10, C11, C12, C13, C14, C15, C16, C17, C18, C2, C3, C4, C5, C6, C7, C8, C9: renamed from C?; footprint (none) -> Capacitor_SMD:C_0603_1608Metric_Pad1.08x0.95mm_HandSolder
- F1: renamed from F?; footprint (none) -> Fuse:Fuse_0603_1608Metric_Pad1.05x0.95mm_HandSolder
- J1: renamed from J?; footprint (none) -> Connector_IDC:IDC-Header_2x25_P2.54mm_Vertical
- J2: renamed from J?; footprint (none) -> Connector_PinHeader_2.00mm:PinHeader_2x20_P2.00mm_Vertical
- JP1: renamed from JP?; footprint (none) -> Resistor_SMD:R_0603_1608Metric_Pad0.98x0.95mm_HandSolder
- R1, R10, R11, R12, R13, R14, R15, R16, R17, R18, R2, R3, R4, R5, R6, R7, R8, R9: renamed from R?; footprint (none) -> Resistor_SMD:R_0603_1608Metric_Pad0.98x0.95mm_HandSolder
- SW1: renamed from SW?; footprint (none) -> Button_Switch_SMD:SW_DIP_SPSTx03_Slide_Omron_A6S-310x_W8.9mm_P2.54mm

Commit message: Update
Parts:
- removed SW1: SW_DIP_x03, Button_Switch_SMD:SW_DIP_SPSTx03_Slide_Omron_A6S-310x_W8.9mm_P2.54mm, symbol Switch:SW_DIP_x03
- added H1, H2: MountingHole, MountingHole:MountingHole_4.3mm_M4, symbol Mechanical:MountingHole
- added J3: Conn_02x03_Odd_Even, Connector_PinHeader_2.54mm:PinHeader_2x03_P2.54mm_Vertical, symbol Connector_Generic:Conn_02x03_Odd_Even
Connections:
- net DB0: now also C1.1, J2.8 (Pin_8), R1.2
- net DB1: now also C2.1, J2.10 (Pin_10), R2.2
- net DB2: now also C3.1, J2.12 (Pin_12), R3.2
- net DB3: now also C4.1, J2.14 (Pin_14), R4.2
- net DB4: now also C5.1, J2.16 (Pin_16), R5.2
- net DB5: now also C6.1, J2.18 (Pin_18), R6.2
- net DB6: now also C7.1, J2.19 (Pin_19), R7.2
- net DB7: now also C8.1, J2.21 (Pin_21), R8.2
- net GND: now also J3.2 (Pin_2), J3.4 (Pin_4), J3.6 (Pin_6)
- net ID_SWITCH1: now also J2.1 (Pin_1), J3.1 (Pin_1)
- net ID_SWITCH2: now also J2.2 (Pin_2), J3.3 (Pin_3)
- net ID_SWITCH3: now also J2.3 (Pin_3), J3.5 (Pin_5)
- net PARITY: now also C9.1, J2.23 (Pin_23), R9.2
- net /ACK: now also C12.1, J2.29 (Pin_29), R12.2
- net /ATN: now also C10.1, J2.26 (Pin_26), R10.2
- net /BSY: now also C11.1, J2.27 (Pin_27), R11.2
- net /C/D: now also C17.1, J2.35 (Pin_35), R17.2
- net /I/O: now also C16.1, J2.34 (Pin_34), R16.2
- net /MSG: now also C14.1, J2.31 (Pin_31), R14.2
- net /REQ: now also C18.1, J2.37 (Pin_37), R18.2
- net /RST: now also C13.1, J2.30 (Pin_30), R13.2
- net /SEL: now also C15.1, J2.33 (Pin_33), R15.2

Commit message: fixes
Parts:
- removed JP1: Jumper_2_Open, Resistor_SMD:R_0603_1608Metric_Pad0.98x0.95mm_HandSolder, symbol Jumper:Jumper_2_Open
- removed R1, R10, R11, R12, R13, R14, R15, R16, R17, R18, R2, R3, R4, R5, R6, R7, R8, R9: R_Small_US, Resistor_SMD:R_0603_1608Metric_Pad0.98x0.95mm_HandSolder, symbol Device:R_Small_US
- added J5: Conn_01x04, Connector_PinHeader_2.54mm:PinHeader_1x04_P2.54mm_Horizontal, symbol Connector_Generic:Conn_01x04
- added RN1, RN2: 4611X-104-221/331L, Resistor_THT:R_Array_SIP11, symbol Device:R_Network_Dividers_x09_SIP
- C1, C10, C11, C12, C13, C14, C15, C16, C17, C18, C2, C3, C4, C5, C6, C7, C8, C9: value C_Small -> 47p; footprint Capacitor_SMD:C_0603_1608Metric_Pad1.08x0.95mm_HandSolder -> Capacitor_SMD:C_0805_2012Metric_Pad1.18x1.45mm_HandSolder; Mouser (none) -> 80-C0805X470J1HACTU
- F1: value Fuse -> 1A; footprint Fuse:Fuse_0603_1608Metric_Pad1.05x0.95mm_HandSolder -> Fuse:Fuse_0805_2012Metric_Pad1.15x1.40mm_HandSolder; Mouser (none) -> 594-MFU0805-FF-1.0
- J1: value Conn_02x25_Odd_Even -> Internal SCSI
- J2: value Conn_02x20_Odd_Even -> X68030 SCSI
Connections:
- net NO_IDEA2 is gone; now on net VCC1: J2.39 (Pin_39), J2.40 (Pin_40)
- net DB0: now also RN1.2 (R1)
- net DB1: now also RN1.3 (R2)
- net DB2: now also RN1.4 (R3)
- net DB3: now also RN1.5 (R4)
- net DB4: now also RN1.6 (R5)
- net DB5: now also RN1.7 (R6)
- net DB6: now also RN1.8 (R7)
- net DB7: now also RN1.9 (R8)
- net GND: now also J2.11 (Pin_11), J2.13 (Pin_13), J2.15 (Pin_15), J2.17 (Pin_17), J2.7 (Pin_7), J2.9 (Pin_9), J5.3 (Pin_3), J5.4 (Pin_4), RN1.11 (COM2), RN2.11 (COM2)
- net PARITY: now also RN1.10 (R9)
- net TMPWR: now also F1.1, RN1.1 (COM1), RN2.1 (COM1)
- net /ACK: now also RN2.4 (R3)
- net /ATN: now also RN2.2 (R1)
- net /BSY: now also RN2.3 (R2)
- net /C/D: now also C16.1, RN2.8 (R7); no longer C17.1
- net /I/O: now also C18.1, RN2.10 (R9); no longer C16.1
- net /MSG: now also RN2.6 (R5)
- net /REQ: now also C17.1, RN2.9 (R8); no longer C18.1
- net /RST: now also RN2.5 (R4)
- net /SEL: now also RN2.7 (R6)
- net at F1.2: now also J2.25 (Pin_25)
- net HDLED: now reaches J2.4 (Pin_4)
- net HDLED: now also J5.2 (Pin_2)
- net ID_SWITCH1 renamed ID0
- net ID_SWITCH2 renamed ID1
- net ID_SWITCH3 renamed ID2
- net NO_IDEA1 renamed VCC1
- net VCC1: now also J5.1 (Pin_1)
- removed net VCC: F1.1, J2.25 (Pin_25)
Other:
- moved on the sheet: F1, H1, H2, J1, J2, J3

Commit message: Update x68030_scsi.kicad_sch
Parts:
- J1: Mouser (none) -> 737-BHR-50-VUA
- J2: Mouser (none) -> 538-87831-4021
Changed lines of the file:
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@@
+			)
+		)
+		(property "Mouser" "737-BHR-50-VUA "
+			(at 81.28 88.9 0)
+			(effects
+				(font
+					(size 1.27 1.27)
+				)
+				(hide yes)
 			)
 		)
@@
 			(at 231.14 85.09 0)
 			(effects
+				(font
+					(size 1.27 1.27)
+				)
+				(hide yes)
+			)
+		)
+		(property "Mouser" "538-87831-4021  "
+			(at 231.14 85.09 0)
+			(effects

Commit message: minor fixes
Parts:
- J3: value Conn_02x03_Odd_Even -> ID_SWITCH
Other:
- moved on the sheet: F1, H1, H2, J1, J2, J3, J5

Commit message: fix stuff
Parts:
- removed J3: ID_SWITCH, Connector_PinHeader_2.54mm:PinHeader_2x03_P2.54mm_Vertical, symbol Connector_Generic:Conn_02x03_Odd_Even
- removed J5: Conn_01x04, Connector_PinHeader_2.54mm:PinHeader_1x04_P2.54mm_Horizontal, symbol Connector_Generic:Conn_01x04
- added JP1: Jumper_2_Small_Bridged, Jumper:SolderJumper-2_P1.3mm_Bridged_Pad1.0x1.5mm, symbol Jumper:Jumper_2_Small_Bridged
- added TP1: EXTERNAL_HDLED1, TestPoint:TestPoint_Pad_1.5x1.5mm, symbol Connector:TestPoint
- added U2: 74LVC1G07, Package_TO_SOT_SMD:SOT-23-5_HandSoldering, symbol 74xGxx:74LVC1G07
Connections:
- net GND: now also U2.3 (GND)
- net VCC1: now also U2.5 (VCC)
- net /BSY: now also JP1.2 (B)
- net HDLED renamed HDLED-
- net HDLED-: now also U2.4
- new net: JP1.1 (A), TP1.1, U2.2
- no-connect marks 1 -> 2

Commit message: updates
Parts:
- removed JP1: Jumper_2_Small_Bridged, Jumper:SolderJumper-2_P1.3mm_Bridged_Pad1.0x1.5mm, symbol Jumper:Jumper_2_Small_Bridged
- removed TP1: EXTERNAL_HDLED1, TestPoint:TestPoint_Pad_1.5x1.5mm, symbol Connector:TestPoint
- removed U2: 74LVC1G07, Package_TO_SOT_SMD:SOT-23-5_HandSoldering, symbol 74xGxx:74LVC1G07
- added J3: Conn_01x02, Connector_JST:JST_XH_B2B-XH-A_1x02_P2.50mm_Vertical, symbol Connector_Generic:Conn_01x02
- added JP1: Jumper_2_Bridged, Jumper:SolderJumper-2_P1.3mm_Bridged_Pad1.0x1.5mm, symbol Jumper:Jumper_2_Bridged
- added JP2: Jumper_2_Open, Jumper:SolderJumper-2_P1.3mm_Open_Pad1.0x1.5mm, symbol Jumper:Jumper_2_Open
- added U1: SN74LVC1G14DBV, Package_TO_SOT_SMD:SOT-23-5, symbol 74xGxx:SN74LVC1G14DBV
Connections:
- net GND: now also U1.3 (GND)
- net HDLED-: now also JP1.2 (B), JP2.2 (B)
- net VCC1: now also U1.5 (VCC)
- new net: J3.2 (Pin_2), JP2.1 (A)
- new net: J3.1 (Pin_1), U1.2
- new net: JP1.1 (A), U1.4
- no-connect marks 2 -> 1
Other:
- moved on the sheet: C1, C10, C11, C12, C13, C14, C15, C16, C17, C18, C2, C3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
